Commit message: move environment files to env_config

File: urdf/robot_event_cam.urdf.xacro (robot description, xacro)
@@ -48,18 +48,18 @@
   </gazebo>
   <!-- Wheel Macro -->
-  <xacro:include filename="$(find ghost)/urdf/omni_wheel.urdf.xacro" />
+  <xacro:include filename="$(find robot_config)/urdf/mecanum_wheel.urdf.xacro" />
   <!-- WHEELS -->
-  <xacro:omni_wheel_250 name="wheel_front_left" parent="agv_base_link">
-    <origin xyz="0.22 0.21 ${-agv_base_height/2-agv_base_lift + agv_wheel_height}" rpy="0 0 0" />
-  </xacro:omni_wheel_250>
-  <xacro:omni_wheel_250 name="wheel_front_right" parent="agv_base_link">
-    <origin xyz="0.22 -0.21 ${-agv_base_height/2-agv_base_lift + agv_wheel_height}" rpy="0 0 0" />
-  </xacro:omni_wheel_250>
-  <xacro:omni_wheel_250 name="wheel_back_left" parent="agv_base_link">
-    <origin xyz="-0.22 0.21 ${-agv_base_height/2-agv_base_lift + agv_wheel_height}" rpy="0 0 0" />
-  </xacro:omni_wheel_250>
-  <xacro:omni_wheel_250 name="wheel_back_right" parent="agv_base_link">
-    <origin xyz="-0.22 -0.21 ${-agv_base_height/2-agv_base_lift + agv_wheel_height}" rpy="0 0 0" />
-  </xacro:omni_wheel_250>
+  <xacro:mecanum_wheel_a name="wheel_front_left" parent="agv_base_link">
+    <origin xyz="0.22 0.21 ${-agv_base_height/2-agv_base_lift + agv_wheel_height}" rpy="${M_PI_2} 0 0" />
+  </xacro:mecanum_wheel_a>
+  <xacro:mecanum_wheel_b name="wheel_front_right" parent="agv_base_link">
+    <origin xyz="0.22 -0.21 ${-agv_base_height/2-agv_base_lift + agv_wheel_height}" rpy="${M_PI_2} 0 0" />
+  </xacro:mecanum_wheel_b>
+  <xacro:mecanum_wheel_b name="wheel_back_left" parent="agv_base_link">
+    <origin xyz="-0.22 0.21 ${-agv_base_height/2-agv_base_lift + agv_wheel_height}" rpy="${M_PI_2} 0 0" />
+  </xacro:mecanum_wheel_b>
+  <xacro:mecanum_wheel_a name="wheel_back_right" parent="agv_base_link">
+    <origin xyz="-0.22 -0.21 ${-agv_base_height/2-agv_base_lift + agv_wheel_height}" rpy="${M_PI_2} 0 0" />
+  </xacro:mecanum_wheel_a>
   <!-- AGV_BASE_LINK -->
   <joint name="base_footprint_agv_base_joint" type="fixed">
