Commit message: added soap_odom.usd

File: urdf/robot.urdf.xacro (robot description, xacro)
@@ -48,5 +48,5 @@
   </gazebo>
   <!-- Wheel Macro -->
-  <xacro:include filename="$(find ghost)/urdf/omni_wheel.urdf.xacro" />
+  <xacro:include filename="$(find config_robot)/urdf/omni_wheel.urdf.xacro" />
   <!-- WHEELS -->
   <xacro:omni_wheel_250 name="wheel_front_left" parent="agv_base_link">

File: urdf/robot2.urdf.xacro (robot description, xacro)
@@ -59,5 +59,5 @@
   </gazebo>
   <!-- Wheel Macro -->
-  <xacro:include filename="$(find ghost)/urdf/omni_wheel.urdf.xacro" />
+  <xacro:include filename="$(find config_robot)/urdf/omni_wheel.urdf.xacro" />
   <!-- WHEELS -->
   <xacro:omni_wheel_250 name="wheel_front_left" parent="agv_base_link">

File: urdf/robot3.urdf.xacro (robot description, xacro)
@@ -58,5 +58,5 @@
   </gazebo>
   <!-- Wheel Macro -->
-  <xacro:include filename="$(find ghost)/urdf/omni_wheel.urdf.xacro" />
+  <xacro:include filename="$(find config_robot)/urdf/omni_wheel.urdf.xacro" />
   <!-- WHEELS -->
   <xacro:omni_wheel_250 name="wheel_front_left" parent="agv_base_link">

File: urdf/robot_dual_cam.urdf.xacro (robot description, xacro)
@@ -48,5 +48,5 @@
   </gazebo>
   <!-- Wheel Macro -->
-  <xacro:include filename="$(find ghost)/urdf/omni_wheel.urdf.xacro" />
+  <xacro:include filename="$(find config_robot)/urdf/omni_wheel.urdf.xacro" />
   <!-- WHEELS -->
   <xacro:omni_wheel_250 name="wheel_front_left" parent="agv_base_link">

File: urdf/robot_event_cam.urdf.xacro (robot description, xacro)
@@ -1,144 +1,61 @@
 <?xml version="1.0"?>
 <robot name="robot" xmlns:xacro="http://ros.org/wiki/xacro">
-  <!-- Defining the colors used in this robot -->
-  <material name="Black">
-    <color rgba="0.0 0.0 0.0 1.0"/>
-  </material>
-  <material name="Red">
-    <color rgba="0.8 0.0 0.0 1.0"/>
-  </material>
-  <material name="White">
-    <color rgba="1.0 1.0 1.0 1.0"/>
-  </material>
-  <material name="Blue">
-    <color rgba="0.0 0.0 0.8 1.0"/>
-  </material>
-  <!-- PROPERTY LIST -->
-  <!--All units in m-kg-s-radians unit system -->
-  <xacro:property name="M_PI" value="3.1415926535897931" />
-  <xacro:property name="M_PI_2" value="1.570796327" />
-  <xacro:property name="DEG_TO_RAD" value="0.017453293" />
-  <!-- box -->
-  <xacro:property name="box_size" value="0.05" />
-  <!-- AGV Base -->
-  <xacro:property name="agv_base_height" value="0.4" />
-  <xacro:property name="agv_base_lift" value="0.025" />
-  <xacro:property name="agv_base_width" value="0.495" />
-  <xacro:property name="agv_base_length" value="0.73" />
-  <xacro:property name="agv_base_mass" value="40" />
-  <xacro:property name="agv_wheel_height" value="0.07825" />
-  <!-- Macro for calculating inertia of cube -->
-  <xacro:macro name="cuboid_inertia" params="m w d h">
-    <inertia  ixx="${m*(h*h+d*d)/12}" ixy = "0" ixz = "0"
-              iyy="${m*(w*w+d*d)/12}" iyz = "0"
-              izz="${m*(w*w+h*h)/12}" />
-  </xacro:macro>
-  <!-- BASE-FOOTPRINT -->
-  <!-- base_footprint is a fictitious link(frame) that is on the ground right below base_link origin -->
-  <link name="base_footprint">
-    <visual>
-        <origin xyz="0 0 0" rpy="0 0 0" />
-        <geometry>
-            <box size="0.001 0.001 0.001" />
-        </geometry>
-    </visual>
-  </link>
-  <gazebo reference="base_footprint">
-    <turnGravityOff>false</turnGravityOff>
-  </gazebo>
-  <!-- Wheel Macro -->
-  <xacro:include filename="$(find robot_config)/urdf/mecanum_wheel.urdf.xacro" />
-  <!-- WHEELS -->
-  <xacro:mecanum_wheel_a name="wheel_front_left" parent="agv_base_link">
-    <origin xyz="0.22 0.21 ${-agv_base_height/2-agv_base_lift + agv_wheel_height}" rpy="${M_PI_2} 0 0" />
-  </xacro:mecanum_wheel_a>
-  <xacro:mecanum_wheel_b name="wheel_front_right" parent="agv_base_link">
-    <origin xyz="0.22 -0.21 ${-agv_base_height/2-agv_base_lift + agv_wheel_height}" rpy="${M_PI_2} 0 0" />
-  </xacro:mecanum_wheel_b>
-  <xacro:mecanum_wheel_b name="wheel_back_left" parent="agv_base_link">
-    <origin xyz="-0.22 0.21 ${-agv_base_height/2-agv_base_lift + agv_wheel_height}" rpy="${M_PI_2} 0 0" />
-  </xacro:mecanum_wheel_b>
-  <xacro:mecanum_wheel_a name="wheel_back_right" parent="agv_base_link">
-    <origin xyz="-0.22 -0.21 ${-agv_base_height/2-agv_base_lift + agv_wheel_height}" rpy="${M_PI_2} 0 0" />
-  </xacro:mecanum_wheel_a>
-  <!-- AGV_BASE_LINK -->
-  <joint name="base_footprint_agv_base_joint" type="fixed">
-    <origin xyz="0 0 ${agv_base_height/2+agv_base_lift}" rpy="0 0 0" />
-    <parent link="base_footprint"/>
-    <child link="agv_base_link" />
-  </joint>
-  <link name="agv_base_link">
-   <inertial>
-     <mass value="${agv_base_mass}" />
-     <origin xyz="0 0 ${-agv_base_height/2-agv_base_lift}" />
-     <cuboid_inertia m="${agv_base_mass}" d="${agv_base_length}" w="${agv_base_width}" h="${agv_base_height}" />
-   </inertial>
-   <visual>
-      <origin xyz="0 0 0" rpy="0 0 0" />
-      <geometry>
-        <box size="${agv_base_length} ${agv_base_width} ${agv_base_height}" />
-      </geometry>
-      <material name="White" />
-    </visual>
-    <collision>
-      <origin xyz="0 0 0" rpy="0 0 0" />
-      <geometry>
-        <box size="${agv_base_length} ${agv_base_width} ${agv_base_height}" />
-      </geometry>
-    </collision>
-  </link>
-  <!-- AGV lidar -->
-  <joint name="base_footprint_lidar_joint" type="fixed">
-	  <origin xyz="0.0 0.0 0.39175" rpy="0 0 ${M_PI}" />
-    <parent link="base_footprint"/>
-    <child link="agv_lidar" />
-  </joint>
-  <link name="agv_lidar">
-    <visual>
-      <origin xyz="0 0 0" rpy="0 0 0" />
-      <geometry>
-        <box size="${box_size} ${box_size} ${box_size}"/>
-      </geometry>
-      <material name="Blue" />
-    </visual>
-  </link>
-  <gazebo reference="agv_lidar">
-    <material>Gazebo/Blue</material>
-    <turnGravityOff>false</turnGravityOff>
-    <sensor type="ray" name="agv_lidar">
-      <pose>${box_size/2} 0 0 0 0 0</pose>
-      <visualize>false</visualize>
-      <update_rate>60</update_rate>
-      <ray>
-        <scan>
-          <horizontal>
-            <samples>721</samples>
-            <resolution>1</resolution>
-            <min_angle>-${M_PI}</min_angle>
-            <max_angle>${M_PI}</max_angle>
-          </horizontal>
-        </scan>
-        <range>
-          <min>0.10</min>
-          <max>20.0</max>
-          <resolution>0.001</resolution>
-        </range>
-      </ray>
-      <plugin name="gazebo_ros_agv_lidar_controller" filename="libgazebo_ros_laser.so">
-        <topicName>/scan</topicName>
-        <frameName>agv_lidar</frameName>
-      </plugin>
-    </sensor>
-  </gazebo>
-  <gazebo>
-    <!-- <plugin name="differential_drive_controller" filename="libgazebo_ros_diff_drive.so"> -->
-    <plugin name="planar_move_controller" filename="libgazebo_ros_planar_move.so">
-      <commandTopic>cmd_vel</commandTopic>
-      <odometryFrame>odom</odometryFrame>
-      <odometryTopic>odom</odometryTopic>
-      <robotBaseFrame>base_footprint</robotBaseFrame>
-      <odometryRate>60.0</odometryRate>
-      <publishTF>true</publishTF>
-    </plugin>
-  </gazebo>
+	<!-- General Macro -->
+	<xacro:include filename="$(find config_robot)/urdf/lib/common.urdf.xacro" />
+	<!-- Wheel Macro -->
+	<xacro:include filename="$(find config_robot)/urdf/lib/wheel/mecanum_wheel.urdf.xacro" />
+	<!-- Lidar Macro -->
+	<xacro:include filename="$(find config_robot)/urdf/lib/sensor/block_lidar.urdf.xacro" />
+	<!-- PROPERTY LIST -->
+	<!--All units in m-kg-s-radians unit system -->
+	<xacro:property name="M_PI_2" value="${pi/2.0}" />
+	<!-- AGV Base -->
+	<xacro:property name="agv_base_height" value="0.4" />
+	<xacro:property name="agv_base_lift" value="0.025" />
+	<xacro:property name="agv_base_width" value="0.495" />
+	<xacro:property name="agv_base_length" value="0.73" />
+	<xacro:property name="agv_base_mass" value="40" />
+	<xacro:property name="agv_wheel_height" value="0.07825" />
+	<!-- BASE-FOOTPRINT -->
+	<!-- base_footprint is a fictitious link(frame) that is on the ground right below base_link origin -->
+	<link name="base_footprint">
+		<xacro:visual_cuboid length="${0.001}" width="${0.001}" height="${0.001}" />
+	</link>
+	<gazebo reference="base_footprint">
+		<turnGravityOff>false</turnGravityOff>
+	</gazebo>
+	<!-- AGV_BASE_LINK -->
+	<joint name="base_footprint_agv_base_joint" type="fixed">
+		<origin xyz="0 0 ${agv_base_height/2+agv_base_lift}" rpy="0 0 0" />
+		<parent link="base_footprint"/>
+		<child link="agv_base_link" />
+	</joint>
+	<link name="agv_base_link">
+		<xacro:inertia_cuboid mass="${agv_base_mass}" d="${agv_base_length}" w="${agv_base_width}"
+													h="${agv_base_height}" xyz="0 0 ${-agv_base_height/2-agv_base_lift}" />
+		<xacro:collision_cuboid length="${agv_base_length}" width="${agv_base_width}" height="${agv_base_height}" />
+		<xacro:visual_cuboid length="${agv_base_length}" width="${agv_base_width}" height="${agv_base_height}" material="White" />
+	</link>
+	<!-- WHEELS -->
+	<xacro:mecanum_wheel_a	name="wheel_front_left" parent="agv_base_link"
+													xyz="0.22 0.21 ${-agv_base_height/2-agv_base_lift + agv_wheel_height}" rpy="${M_PI_2} 0 0" />
+	<xacro:mecanum_wheel_b	name="wheel_front_right" parent="agv_base_link"
+													xyz="0.22 -0.21 ${-agv_base_height/2-agv_base_lift + agv_wheel_height}" rpy="${-M_PI_2} 0 0" />
+	<xacro:mecanum_wheel_b	name="wheel_back_left" parent="agv_base_link"
+													xyz="-0.22 0.21 ${-agv_base_height/2-agv_base_lift + agv_wheel_height}" rpy="${M_PI_2} 0 0" />
+	<xacro:mecanum_wheel_a	name="wheel_back_right" parent="agv_base_link"
+													xyz="-0.22 -0.21 ${-agv_base_height/2-agv_base_lift + agv_wheel_height}" rpy="${-M_PI_2} 0 0" />
+	<!-- AGV lidar -->
+	<xacro:block_lidar name="agv_lidar" parent="base_footprint" xyz="0.0 0.0 0.45" rpy="0 0 ${pi}" />
+	<gazebo>
+		<!-- <plugin name="differential_drive_controller" filename="libgazebo_ros_diff_drive.so"> -->
+		<plugin name="planar_move_controller" filename="libgazebo_ros_planar_move.so">
+			<commandTopic>cmd_vel</commandTopic>
+			<odometryFrame>odom</odometryFrame>
+			<odometryTopic>odom</odometryTopic>
+			<robotBaseFrame>base_footprint</robotBaseFrame>
+			<odometryRate>60.0</odometryRate>
+			<publishTF>true</publishTF>
+		</plugin>
+	</gazebo>
 </robot>

File: urdf/robot_no_odom.urdf.xacro (robot description, xacro)
@@ -48,5 +48,5 @@
   </gazebo>
   <!-- Wheel Macro -->
-  <xacro:include filename="$(find ghost)/urdf/omni_wheel.urdf.xacro" />
+  <xacro:include filename="$(find config_robot)/urdf/omni_wheel.urdf.xacro" />
   <!-- WHEELS -->
   <xacro:omni_wheel_250 name="wheel_front_left" parent="agv_base_link">

File: urdf/robot_v0.urdf.xacro (robot description, xacro)
@@ -52,5 +52,5 @@
   </gazebo>
   <!-- Wheel Macro -->
-  <xacro:include filename="$(find ghost)/urdf/omni_wheel.urdf.xacro" />
+  <xacro:include filename="$(find config_robot)/urdf/omni_wheel.urdf.xacro" />
   <!-- WHEELS -->
   <xacro:omni_wheel_250 name="wheel_front_left" parent="agv_base_link">

File: urdf/robot_v1.urdf.xacro (robot description, xacro)
@@ -52,5 +52,5 @@
   </gazebo>
   <!-- Wheel Macro -->
-  <xacro:include filename="$(find ghost)/urdf/omni_wheel.urdf.xacro" />
+  <xacro:include filename="$(find config_robot)/urdf/omni_wheel.urdf.xacro" />
   <!-- WHEELS -->
   <xacro:omni_wheel_250 name="wheel_front_left" parent="agv_base_link">
