Commit message: updated robots urdf

File: urdf/diff_wheelbarrow.urdf.xacro (robot description, xacro)
@@ -1,9 +1,13 @@
 <?xml version="1.0"?>
-<robot name="robot" xmlns:xacro="http://ros.org/wiki/xacro">
+<robot name="wheelbarrow" xmlns:xacro="http://ros.org/wiki/xacro">
 	<!-- General Macro -->
 	<xacro:include filename="$(find config_robot)/urdf/lib/common.urdf.xacro" />
 	<!-- Wheel Macro -->
 	<xacro:include filename="$(find config_robot)/urdf/lib/wheel/wheel.urdf.xacro" />
-	<xacro:include filename="$(find config_robot)/urdf/lib/wheel/swivel_caster.urdf.xacro" />
+	<xacro:include filename="$(find config_robot)/urdf/lib/wheel/caster_wheel.urdf.xacro" />
+	<!-- IMU Macro -->
+	<xacro:include filename="$(find config_robot)/urdf/lib/sensor/block_imu.urdf.xacro" />
+	<!-- Lidar Macro -->
+	<xacro:include filename="$(find config_robot)/urdf/lib/sensor/block_lidar.urdf.xacro" />
 	<!-- PROPERTY LIST -->
 	<!--All units in m-kg-s-radians unit system -->
@@ -18,9 +22,5 @@
 	<!-- BASE-FOOTPRINT -->
 	<!-- base_footprint is a fictitious link(frame) that is on the ground right below base_link origin -->
-	<link name="base_footprint">
-		<xacro:inertia_cuboid  mass="${agv_base_mass}" d="${0.001}" w="${0.001}" h="${0.001}" xyz="0 0 0" />
-		<xacro:collision_cuboid length="${0.001}" width="${0.001}" height="${0.001}" />
-		<xacro:visual_cuboid length="${0.001}" width="${0.001}" height="${0.001}" material="White" />
-	</link>
+	<link name="base_footprint"/>
 	<!-- AGV_BASE_LINK -->
 	<joint name="agv_base_joint" type="fixed">
@@ -31,6 +31,5 @@
 	<link name="agv_base_link">
 		<!-- body -->
-		<xacro:inertia_cuboid mass="${agv_base_mass}" d="${agv_base_length}" w="${agv_base_width}"
-													h="${agv_base_height}" xyz="0 0 ${-agv_base_height/2-agv_base_lift}" />
+		<xacro:inertia_cuboid mass="${agv_base_mass}" d="${agv_base_length}" w="${agv_base_width}" h="${agv_base_height}" />
 		<xacro:collision_cuboid length="${agv_base_length}" width="${agv_base_width}" height="${agv_base_height}" />
 		<xacro:visual_cuboid length="${agv_base_length}" width="${agv_base_width}" height="${agv_base_height}" material="White" />
@@ -77,4 +76,6 @@
 		<xacro:visual_cylinder radius="${radius}" length="${handle_length}" xyz="${handle_xyz}" rpy="${handle_rpy}" />
 	</link>
+	<!-- IMU -->
+	<xacro:block_imu name="imu_link" parent="agv_base_link" xyz="0.0 0.0 0.0" rpy="0.0 0.0 0.0" />
 	<!-- WHEEL_CENTER_LINK -->
 	<joint name="wheel_center_joint" type="fixed">
@@ -89,7 +90,7 @@
 	<xacro:wheel	name="wheel_right" parent="agv_base_link"
 													xyz="-0.22 -0.15 ${-agv_base_height/2-agv_base_lift + agv_wheel_height}" rpy="${-M_PI_2} 0 0" />
-	<xacro:swivel_caster	name="swivel_caster_left" parent="agv_base_link"
-													xyz="0.22 0.15 ${-agv_base_height/2-agv_base_lift + agv_wheel_height}" rpy="${M_PI_2} 0 0" />
-	<xacro:swivel_caster	name="swivel_caster_right" parent="agv_base_link"
-													xyz="0.22 -0.15 ${-agv_base_height/2-agv_base_lift + agv_wheel_height}" rpy="${-M_PI_2} 0 0" />
+	<xacro:caster_wheel	name="caster_left" parent="agv_base_link"
+													xyz="0.22 0.15 ${-agv_base_height/2-agv_base_lift + agv_wheel_height}" rpy="0 ${pi} 0" />
+	<xacro:caster_wheel	name="caster_right" parent="agv_base_link"
+													xyz="0.22 -0.15 ${-agv_base_height/2-agv_base_lift + agv_wheel_height}" rpy="0 ${pi} 0" />
 </robot>

File: urdf/lib/common.urdf.xacro (robot description, xacro)
@@ -1,4 +1,4 @@
 <?xml version="1.0"?>
-<robot name="common" xmlns:xacro="http://ros.org/wiki/xacro">
+<robot xmlns:xacro="http://www.ros.org/wiki/xacro">
 	<material name="Black">
 		<color rgba="0.0 0.0 0.0 1.0"/>

File: urdf/lib/sensor/block_camera.urdf.xacro (robot description, xacro)
@@ -1,8 +1,8 @@
 <?xml version="1.0"?>
-<robot name="camera" xmlns:xacro="http://ros.org/wiki/xacro">
+<robot xmlns:xacro="http://www.ros.org/wiki/xacro">
 	<!-- camera -->
 	<xacro:property name="cam_size" value="0.05" />
 	<xacro:macro name="camera_gazebo" params="name">
-		<gazebo reference="ideal_${name}">
+		<gazebo reference="${name}">
 			<sensor type="camera" name="${name}">
 				<update_rate>30</update_rate>
@@ -26,5 +26,5 @@
 				<plugin name="camera_controller" filename="libgazebo_ros_camera.so">
 					<imageTopicName>image_raw</imageTopicName>
-					<frameName>ideal_${name}</frameName>
+					<frameName>${name}</frameName>
 					<alwaysOn>true</alwaysOn>
 					<updateRate>1.0</updateRate>
@@ -55,5 +55,5 @@
 	</xacro:macro>
 	<xacro:macro name="block_camera" params="name parent xyz:='0 0 0' rpy:='0 0 0'">
-		<joint name="ideal_${name}_joint" type="fixed">
+		<joint name="${name}_joint" type="fixed">
 			<origin xyz="${xyz}" rpy="${rpy}" />
 			<parent link="${parent}" />

File: urdf/lib/sensor/block_imu.urdf.xacro (robot description, xacro)
@@ -1,10 +1,10 @@
 <?xml version="1.0"?>
-<robot name="lidar" xmlns:xacro="http://ros.org/wiki/xacro">
+<robot xmlns:xacro="http://www.ros.org/wiki/xacro">
 	<!-- lidar -->
-	<xacro:property name="imu_size" value="0.041" />
+	<xacro:property name="imu_size" value="0.001" />
 	<xacro:macro name="imu_gazebo" params="name">
 		<gazebo reference="${name}">
 			<gravity>true</gravity>
-			<sensor name="imu_sensor" type="imu">
+			<sensor type="imu" name="${name}">
 				<always_on>true</always_on>
 				<update_rate>500</update_rate>
@@ -32,5 +32,5 @@
 		</joint>
 		<link name="${name}">
-			<xacro:inertia_cuboid mass="0.1" d="${imu_size}" w="${imu_size}" h="${imu_size}" />
+			<xacro:inertia_cuboid mass="0.01" d="${imu_size}" w="${imu_size}" h="${imu_size}" />
 			<xacro:collision_cuboid length="${imu_size}" width="${imu_size}" height="${imu_size}" />
 			<xacro:visual_cuboid length="${imu_size}" width="${imu_size}" height="${imu_size}"  material="Blue" />

File: urdf/lib/sensor/block_lidar.urdf.xacro (robot description, xacro)
@@ -1,11 +1,11 @@
 <?xml version="1.0"?>
-<robot name="lidar" xmlns:xacro="http://ros.org/wiki/xacro">
+<robot xmlns:xacro="http://www.ros.org/wiki/xacro">
 	<!-- lidar -->
-	<xacro:property name="lidar_size" value="0.041" />
-	<xacro:macro name="imu_gazebo" params="name">
+	<xacro:property name="lidar_size" value="0.01" />
+	<xacro:macro name="lidar_gazebo" params="name">
 		<gazebo reference="${name}">
 			<sensor type="ray" name="${name}">
-				<pose>${lidar_size/2} 0 0 0 0 0</pose>
-				<visualize>false</visualize>
+				<pose>0 0 0 0 0 0</pose>
+				<visualize>true</visualize>
 				<update_rate>40</update_rate>
 				<ray>
@@ -14,16 +14,25 @@
 							<samples>720</samples>
 							<resolution>1</resolution>
-							<min_angle>${-M_PI}</min_angle>
-							<max_angle>${M_PI}</max_angle>
+							<min_angle>${-pi}</min_angle>
+							<max_angle>${pi}</max_angle>
 						</horizontal>
 					</scan>
+					<noise>
+						<type>gaussian</type>
+						<!-- Noise parameters based on published spec for Hokuyo laser
+							achieving "+-30mm" accuracy at range < 10m.  A mean of 0.0m and
+							stddev of 0.01m will put 99.7% of samples within 0.03m of the true
+							reading. -->
+						<mean>0.0</mean>
+						<stddev>0.01</stddev>
+					</noise>
 					<range>
-						<min>0.15</min>
-						<max>12.0</max>
+						<min>0.45</min>
+						<max>100.0</max>
 						<resolution>0.001</resolution>
 					</range>
 				</ray>
 				<plugin name="gazebo_ros_base_laser_controller" filename="libgazebo_ros_laser.so">
-					<topicName>/scan_${name}</topicName>
+					<topicName>/scan</topicName>
 					<frameName>${name}</frameName>
 				</plugin>
@@ -51,7 +60,7 @@
 		</joint>
 		<link name="${name}">
-			<xacro:inertia_cuboid mass="0.1" d="${lidar_size}" w="${lidar_size}" h="${lidar_size}" />
+			<!-- <xacro:inertia_cuboid mass="0.1" d="${lidar_size}" w="${lidar_size}" h="${lidar_size}" />
 			<xacro:collision_cuboid length="${lidar_size}" width="${lidar_size}" height="${lidar_size}" />
-			<xacro:visual_cuboid length="${lidar_size}" width="${lidar_size}" height="${lidar_size}"  material="Blue" />
+			<xacro:visual_cuboid length="${lidar_size}" width="${lidar_size}" height="${lidar_size}"  material="Blue" /> -->
 		</link>
 	</xacro:macro>

File: urdf/lib/wheel/mecanum_wheel.urdf.xacro (robot description, xacro)
@@ -1,5 +1,5 @@
 <?xml version="1.0"?>
-<robot name="wheel" xmlns:xacro="http://ros.org/wiki/xacro">
-  <xacro:macro name="roller" params="wheel_name num roller_angle N radius roller_bottom_offset damping:=1000000.0">
+<robot xmlns:xacro="http://www.ros.org/wiki/xacro">
+  <xacro:macro name="roller" params="wheel_name num roller_angle N radius roller_bottom_offset">
 		<xacro:property name="axis_offset" value="${roller_bottom_offset + radius}"/>
 		<xacro:property name="angle" value="${2*num*N*pi}"/>
@@ -9,5 +9,5 @@
 			<parent link="${wheel_name}"/>
 			<child link="roller_${wheel_name}_${num}"/>
-			<dynamics damping="${damping}" friction="0.0" />
+			<dynamics damping="0.01" friction="0.0" />
 		</joint>
 		<link name="roller_${wheel_name}_${num}">
@@ -17,5 +17,5 @@
 		</link>
 	</xacro:macro>
-	<xacro:macro name="mecanum_wheel" params="wheel_name parent roller_angle xyz:='0 0 0' rpy:='0 0 0' damping:=1000000.0">
+	<xacro:macro name="mecanum_wheel" params="wheel_name parent roller_angle xyz:='0 0 0' rpy:='0 0 0'">
 		<xacro:property name="wheel_radius" value="0.07825"/>
 		<xacro:property name="core_radius" value="${wheel_radius * 0.76}"/>
@@ -29,5 +29,5 @@
 			<parent link="${parent}" />
 			<child link="${wheel_name}" />
-			<dynamics damping="${damping}" friction="0.0" />
+			<dynamics damping="0.01" friction="0.0" />
 		</joint>
 		<link name="${wheel_name}">

File: urdf/lib/wheel/omni_wheel.urdf.xacro (robot description, xacro)
@@ -1,5 +1,5 @@
 <?xml version="1.0"?>
-<robot name="wheel" xmlns:xacro="http://ros.org/wiki/xacro">
-  <xacro:macro name="roller" params="wheel_name num radius visual_axis_offset roller_bottom_offset side damping:=1000000.0">
+<robot xmlns:xacro="http://www.ros.org/wiki/xacro">
+  <xacro:macro name="roller" params="wheel_name num radius visual_axis_offset roller_bottom_offset side">
 		<!-- Radius of the sphere used for the roller -->
 		<!-- <xacro:property name="radius" value="${radius}"/> -->
@@ -16,5 +16,5 @@
 			<parent link="${wheel_name}"/>
 			<child link="roller_${wheel_name}_${side}_${num}"/>
-			<dynamics damping="${damping}" friction="0.0" />
+			<dynamics damping="1.0" friction="0.0" />
 		</joint>
 		<link name="roller_${wheel_name}_${side}_${num}">
@@ -24,5 +24,5 @@
 		</link>
 	</xacro:macro>
-	<xacro:macro name="omni_wheel" params="name parent xyz:='0 0 0' rpy:='0 0 0' damping:=1000000.0">
+	<xacro:macro name="omni_wheel" params="name parent xyz:='0 0 0' rpy:='0 0 0'">
 		<xacro:property name="radius" value="0.07825"/>
 		<xacro:property name="length" value="0.085"/>
@@ -34,5 +34,5 @@
 			<parent link="${parent}" />
 			<child link="${name}" />
-			<dynamics damping="${damping}" friction="0.0" />
+			<dynamics damping="1.0" friction="0.0" />
 		</joint>
 		<link name="${name}">

File: urdf/lib/wheel/wheel.urdf.xacro (robot description, xacro)
@@ -1,5 +1,5 @@
 <?xml version="1.0"?>
-<robot name="wheel" xmlns:xacro="http://ros.org/wiki/xacro">
-	<xacro:macro name="wheel" params="name parent xyz:='0 0 0' rpy:='0 0 0' damping:=1000000.0">
+<robot xmlns:xacro="http://www.ros.org/wiki/xacro">
+	<xacro:macro name="wheel" params="name parent xyz:='0 0 0' rpy:='0 0 0'">
 		<xacro:property name="radius" value="0.07825"/>
 		<xacro:property name="length" value="0.085"/>
@@ -11,5 +11,5 @@
 			<parent link="${parent}" />
 			<child link="${name}" />
-			<dynamics damping="${damping}" friction="0.0" />
+			<dynamics damping="1.0" friction="0.0" />
 		</joint>
 		<link name="${name}">
