Commit message: added new robot model

File: urdf/diff_base.gazebo.xacro (robot description, xacro)
@@ -1,4 +1,4 @@
 <?xml version="1.0"?>
-<robot name="wheelbarrow" xmlns:xacro="http://ros.org/wiki/xacro">
+<robot name="diff_base" xmlns:xacro="http://ros.org/wiki/xacro">
 	<!-- Robot Macro -->
 	<xacro:include filename="$(find config_robot)/urdf/diff_base.urdf.xacro" />
@@ -7,5 +7,5 @@
 	</gazebo>
 	<!-- IMU gazebo simulation -->
-	<xacro:imu_gazebo name="imu_link" />
+	<xacro:imu_gazebo name="center_imu" />
 	<!-- IMU gazebo simulation -->
 	<xacro:lidar_gazebo name="lidar_link" />
@@ -22,11 +22,11 @@
       <publishWheelJointState>true</publishWheelJointState>
       <legacyMode>false</legacyMode>
-      <updateRate>30</updateRate>
+      <updateRate>50</updateRate>
       <leftJoint>wheel_left_joint</leftJoint>
       <rightJoint>wheel_right_joint</rightJoint>
       <wheelSeparation>0.3</wheelSeparation>
       <wheelDiameter>0.1565</wheelDiameter>
-      <wheelAcceleration>1</wheelAcceleration>
-      <wheelTorque>10</wheelTorque>
+      <wheelAcceleration>20</wheelAcceleration>
+      <wheelTorque>50</wheelTorque>
       <rosDebugLevel>na</rosDebugLevel>
   	</plugin>
@@ -38,5 +38,5 @@
     <kd>1.0</kd>
     <minDepth>0.001</minDepth>
-    <maxVel>0.1</maxVel>
+    <maxVel>10.0</maxVel>
     <fdir1>1 0 0</fdir1>
     <material>Gazebo/FlatBlack</material>
@@ -48,5 +48,5 @@
     <kd>1.0</kd>
     <minDepth>0.001</minDepth>
-    <maxVel>0.1</maxVel>
+    <maxVel>10.0</maxVel>
     <fdir1>1 0 0</fdir1>
     <material>Gazebo/FlatBlack</material>
@@ -58,5 +58,5 @@
     <kd>1.0</kd>
     <minDepth>0.001</minDepth>
-    <maxVel>1.0</maxVel>
+    <maxVel>10.0</maxVel>
 		<fdir1>1 0 0</fdir1>
     <material>Gazebo/FlatBlack</material>
@@ -68,5 +68,5 @@
     <kd>1.0</kd>
     <minDepth>.001</minDepth>
-    <maxVel>1.0</maxVel>
+    <maxVel>10.0</maxVel>
 		<fdir1>1 0 0</fdir1>
     <material>Gazebo/FlatBlack</material>
@@ -78,5 +78,5 @@
     <kd>1.0</kd>
     <minDepth>0.001</minDepth>
-    <maxVel>1.0</maxVel>
+    <maxVel>10.0</maxVel>
 		<fdir1>1 0 0</fdir1>
     <material>Gazebo/FlatBlack</material>
@@ -88,5 +88,5 @@
     <kd>1.0</kd>
     <minDepth>.001</minDepth>
-    <maxVel>1.0</maxVel>
+    <maxVel>10.0</maxVel>
 		<fdir1>1 0 0</fdir1>
     <material>Gazebo/FlatBlack</material>

File: urdf/diff_base.urdf.xacro (robot description, xacro)
@@ -1,4 +1,4 @@
 <?xml version="1.0"?>
-<robot name="wheelbarrow" xmlns:xacro="http://ros.org/wiki/xacro">
+<robot name="diff_base" xmlns:xacro="http://ros.org/wiki/xacro">
 	<!-- General Macro -->
 	<xacro:include filename="$(find config_robot)/urdf/lib/common.urdf.xacro" />
@@ -36,5 +36,5 @@
 	</link>
 	<!-- IMU -->
-	<xacro:block_imu name="imu_link" parent="agv_base_link" xyz="0.0 0.0 0.0" rpy="0.0 0.0 0.0" />
+	<xacro:block_imu name="center_imu" parent="agv_base_link" xyz="0.0 0.0 0.0" rpy="0.0 0.0 0.0" />
 	<!-- Lidar -->
 	<xacro:block_imu name="lidar_link" parent="agv_base_link" xyz="0.0 0.0 0.025" rpy="0.0 0.0 0.0" />

File: urdf/lib/sensor/block_imu.urdf.xacro (robot description, xacro)
@@ -3,20 +3,20 @@
 	<!-- lidar -->
 	<xacro:property name="imu_size" value="0.001" />
-	<xacro:macro name="imu_gazebo" params="name">
+	<xacro:macro name="imu_gazebo" params="name hz:=100.0">
 		<gazebo reference="${name}">
 			<gravity>true</gravity>
 			<sensor type="imu" name="${name}">
 				<always_on>true</always_on>
-				<update_rate>500</update_rate>
+				<update_rate>${hz}</update_rate>
 				<visualize>true</visualize>
 				<topic>__default_topic__</topic>
 				<plugin filename="libgazebo_ros_imu_sensor.so" name="imu_plugin">
-					<topicName>imu</topicName>
-					<bodyName>imu_link</bodyName>
-					<updateRateHZ>100.0</updateRateHZ>
+					<topicName>${name}</topicName>
+					<bodyName>${name}</bodyName>
+					<updateRateHZ>${hz}</updateRateHZ>
 					<gaussianNoise>0.0</gaussianNoise>
 					<xyzOffset>0 0 0</xyzOffset>
 					<rpyOffset>0 0 0</rpyOffset>
-					<frameName>imu_link</frameName>
+					<frameName>${name}</frameName>
 					<initialOrientationAsReference>false</initialOrientationAsReference>
 				</plugin>
@@ -25,4 +25,16 @@
 		</gazebo>
 	</xacro:macro>
+	<!-- <xacro:macro name="imu_gazebo" params="name">
+		<gazebo>
+		  <plugin name="imu_plugin" filename="libgazebo_ros_imu.so">
+		    <alwaysOn>true</alwaysOn>
+		    <bodyName>"${name}"</bodyName>
+		    <topicName>"${name}"</topicName>
+		    <serviceName>imu_service</serviceName>
+		    <gaussianNoise>0.0</gaussianNoise>
+		    <updateRate>20.0</updateRate>
+		  </plugin>
+		</gazebo>
+  </xacro:macro> -->
 	<xacro:macro name="block_imu" params="name parent xyz:='0 0 0' rpy:='0 0 0'">
 		<joint name="${name}_joint" type="fixed">

File: urdf/lib/wheel/caster_wheel.urdf.xacro (robot description, xacro)
@@ -9,5 +9,5 @@
 			<parent link="${parent}" />
 			<child link="${name}_planner" />
-			<dynamics damping="0.01" friction="0.0" />
+			<dynamics damping="0.01" friction="0.2" />
 		</joint>
 		<link name="${name}_planner">
