Commit message: added diff wheelbarrow

File: urdf/lib/wheel/mecanum_wheel.urdf.xacro (robot description, xacro)
@@ -31,5 +31,5 @@
 			<dynamics damping="1000000.0" friction="0.0" />
 		</joint>
-		<link name="${wheel_name}" type="wheel">
+		<link name="${wheel_name}">
 			<xacro:inertia_cylinder mass="${mass}" radius="${core_radius}" length="${length}" />
 			<xacro:collision_cylinder radius="${core_radius}" length="${length}" />

File: urdf/lib/wheel/omni_wheel.urdf.xacro (robot description, xacro)
@@ -36,5 +36,5 @@
 			<dynamics damping="1000000.0" friction="0.0" />
 		</joint>
-		<link name="${name}" type="wheel">
+		<link name="${name}">
 			<xacro:inertia_cylinder mass="${mass}" radius="${radius}" length="${length}" />
 			<xacro:collision_cylinder radius="${radius}" length="${length}" />

File: urdf/lib/wheel/wheel.urdf.xacro (robot description, xacro)
@@ -1,5 +1,5 @@
 <?xml version="1.0"?>
 <robot name="wheel" xmlns:xacro="http://ros.org/wiki/xacro">
-	<xacro:macro name="wheel" params="name parent *origin">
+	<xacro:macro name="wheel" params="name parent xyz:='0 0 0' rpy:='0 0 0'">
 		<xacro:property name="radius" value="0.07825"/>
 		<xacro:property name="length" value="0.085"/>
@@ -7,10 +7,10 @@
 		<joint name="${name}_joint" type="continuous">
 			<axis xyz="0 0 1" />
-			<xacro:insert_block name="origin" />
+			<origin xyz="${xyz}" rpy="${rpy}" />
 			<parent link="${parent}" />
 			<child link="${name}" />
 			<dynamics damping="1000000.0" friction="0.0" />
 		</joint>
-		<link name="${name}" type="wheel">
+		<link name="${name}">
 			<xacro:inertia_cylinder mass="${mass}" radius="${radius}" length="${length}" />
 			<xacro:collision_cylinder radius="${radius}" length="${length}" />
