Commit message: updated wheel

File: urdf/lib/wheel/wheel.urdf.xacro (robot description, xacro)
@@ -4,4 +4,5 @@
 		<xacro:property name="radius" value="0.07825"/>
 		<xacro:property name="length" value="0.085"/>
+		<xacro:property name="rho" value="1046.3516"/>
 		<xacro:property name="mass" value="2.1"/>
 		<joint name="${name}_joint" type="continuous">
@@ -13,6 +14,8 @@
 		</joint>
 		<link name="${name}">
-			<xacro:inertia_cylinder mass="${mass}" radius="${radius}" length="${length}" />
-			<xacro:collision_cylinder radius="${radius}" length="${length}" />
+			<!-- Make the wheel has one point contact to the ground -->
+			<xacro:inertia_sphere rho="${rho}" radius="${radius}" />
+			<xacro:collision_sphere radius="${radius}" />
+			<!-- Show as a cylinder -->
 			<xacro:visual_cylinder radius="${radius}" length="${length}" />
 		</link>
