Commit message: prepare update for support omniverse + gazebo

File: urdf/lib/common.urdf.xacro (robot description, xacro)
@@ -25,11 +25,11 @@
   <!-- Macro for calculating inertia of sphere -->
 	<xacro:macro name="inertia_sphere" params="radius rho:=1000 xyz:='0 0 0' rpy:='0 0 0'">
-		<xacro:property name="m" value="${4/3*rho*pi*radius**3}"/>
+		<xacro:property name="mass" value="${4/3*rho*pi*radius**3}"/>
 		<inertial>
 			<origin xyz="${xyz}" rpy="${rpy}"/>
-			<mass value="${m}"/>
-			<inertia	ixx="${(2/5*m)*(radius**2)}" ixy="0" ixz="0"
-								iyy="${(2/5*m)*(radius**2)}"  iyz="0"
-								izz="${(2/5*m)*(radius**2)}" />
+			<mass value="${mass}"/>
+			<inertia	ixx="${(2/5*mass)*(radius**2)}" ixy="0" ixz="0"
+								iyy="${(2/5*mass)*(radius**2)}"  iyz="0"
+								izz="${(2/5*mass)*(radius**2)}" />
 		</inertial>
 	</xacro:macro>
@@ -38,4 +38,5 @@
 	<inertial>
 		<origin xyz="${xyz}" rpy="${rpy}"/>
+		<mass value="${mass}"/>
 		<inertia	ixx="${mass*(h*h+d*d)/12}" ixy = "0" ixz = "0"
 							iyy="${mass*(w*w+d*d)/12}" iyz = "0"

File: urdf/lib/sensor/block_lidar.urdf.xacro (robot description, xacro)
@@ -3,30 +3,30 @@
 	<!-- lidar -->
 	<xacro:property name="lidar_size" value="0.041" />
-	<xacro:macro name="lidar_gazebo" params="name">
+	<xacro:macro name="imu_gazebo" params="name">
 		<gazebo reference="${name}">
 			<sensor type="ray" name="${name}">
-			<pose>${lidar_size/2} 0 0 0 0 0</pose>
-			<visualize>false</visualize>
-			<update_rate>40</update_rate>
-			<ray>
-				<scan>
-					<horizontal>
-						<samples>720</samples>
-						<resolution>1</resolution>
-						<min_angle>${-M_PI}</min_angle>
-						<max_angle>${M_PI}</max_angle>
-					</horizontal>
-				</scan>
-				<range>
-					<min>0.15</min>
-					<max>12.0</max>
-					<resolution>0.001</resolution>
-				</range>
-			</ray>
-			<plugin name="gazebo_ros_base_laser_controller" filename="libgazebo_ros_laser.so">
-				<topicName>/scan_${name}</topicName>
-				<frameName>${name}</frameName>
-			</plugin>
-    </sensor>
+				<pose>${lidar_size/2} 0 0 0 0 0</pose>
+				<visualize>false</visualize>
+				<update_rate>40</update_rate>
+				<ray>
+					<scan>
+						<horizontal>
+							<samples>720</samples>
+							<resolution>1</resolution>
+							<min_angle>${-M_PI}</min_angle>
+							<max_angle>${M_PI}</max_angle>
+						</horizontal>
+					</scan>
+					<range>
+						<min>0.15</min>
+						<max>12.0</max>
+						<resolution>0.001</resolution>
+					</range>
+				</ray>
+				<plugin name="gazebo_ros_base_laser_controller" filename="libgazebo_ros_laser.so">
+					<topicName>/scan_${name}</topicName>
+					<frameName>${name}</frameName>
+				</plugin>
+    	</sensor>
 		<!--<material>Gazebo/Blue</material>
 		<gravity>true</gravity>

File: urdf/lib/wheel/mecanum_wheel.urdf.xacro (robot description, xacro)
@@ -1,5 +1,5 @@
 <?xml version="1.0"?>
 <robot name="wheel" xmlns:xacro="http://ros.org/wiki/xacro">
-  <xacro:macro name="roller" params="wheel_name num roller_angle N radius roller_bottom_offset">
+  <xacro:macro name="roller" params="wheel_name num roller_angle N radius roller_bottom_offset damping:=1000000.0">
 		<xacro:property name="axis_offset" value="${roller_bottom_offset + radius}"/>
 		<xacro:property name="angle" value="${2*num*N*pi}"/>
@@ -9,5 +9,5 @@
 			<parent link="${wheel_name}"/>
 			<child link="roller_${wheel_name}_${num}"/>
-			<dynamics damping="1000000.0" friction="0.0" />
+			<dynamics damping="${damping}" friction="0.0" />
 		</joint>
 		<link name="roller_${wheel_name}_${num}">
@@ -17,5 +17,5 @@
 		</link>
 	</xacro:macro>
-	<xacro:macro name="mecanum_wheel" params="wheel_name parent roller_angle xyz:='0 0 0' rpy:='0 0 0'">
+	<xacro:macro name="mecanum_wheel" params="wheel_name parent roller_angle xyz:='0 0 0' rpy:='0 0 0' damping:=1000000.0">
 		<xacro:property name="wheel_radius" value="0.07825"/>
 		<xacro:property name="core_radius" value="${wheel_radius * 0.76}"/>
@@ -29,5 +29,5 @@
 			<parent link="${parent}" />
 			<child link="${wheel_name}" />
-			<dynamics damping="1000000.0" friction="0.0" />
+			<dynamics damping="${damping}" friction="0.0" />
 		</joint>
 		<link name="${wheel_name}">

File: urdf/lib/wheel/omni_wheel.urdf.xacro (robot description, xacro)
@@ -1,5 +1,5 @@
 <?xml version="1.0"?>
 <robot name="wheel" xmlns:xacro="http://ros.org/wiki/xacro">
-  <xacro:macro name="roller" params="wheel_name num radius visual_axis_offset roller_bottom_offset side">
+  <xacro:macro name="roller" params="wheel_name num radius visual_axis_offset roller_bottom_offset side damping:=1000000.0">
 		<!-- Radius of the sphere used for the roller -->
 		<!-- <xacro:property name="radius" value="${radius}"/> -->
@@ -16,5 +16,5 @@
 			<parent link="${wheel_name}"/>
 			<child link="roller_${wheel_name}_${side}_${num}"/>
-			<dynamics damping="1000000.0" friction="0.0" />
+			<dynamics damping="${damping}" friction="0.0" />
 		</joint>
 		<link name="roller_${wheel_name}_${side}_${num}">
@@ -24,5 +24,5 @@
 		</link>
 	</xacro:macro>
-	<xacro:macro name="omni_wheel" params="name parent xyz:='0 0 0' rpy:='0 0 0'">
+	<xacro:macro name="omni_wheel" params="name parent xyz:='0 0 0' rpy:='0 0 0' damping:=1000000.0">
 		<xacro:property name="radius" value="0.07825"/>
 		<xacro:property name="length" value="0.085"/>
@@ -34,5 +34,5 @@
 			<parent link="${parent}" />
 			<child link="${name}" />
-			<dynamics damping="1000000.0" friction="0.0" />
+			<dynamics damping="${damping}" friction="0.0" />
 		</joint>
 		<link name="${name}">

File: urdf/lib/wheel/swivel_caster.urdf.xacro (robot description, xacro)
@@ -1,5 +1,5 @@
 <?xml version="1.0"?>
 <robot name="swivel_caster" xmlns:xacro="http://ros.org/wiki/xacro">
-	<xacro:macro name="swivel_caster" params="name parent xyz:='0 0 0' rpy:='0 0 0'">
+	<xacro:macro name="swivel_caster" params="name parent xyz:='0 0 0' rpy:='0 0 0' damping:=1000000.0">
 		<xacro:property name="radius" value="0.07825"/>
 		<xacro:property name="rho" value="1046.3516"/>
@@ -9,5 +9,5 @@
 			<parent link="${parent}" />
 			<child link="${name}" />
-			<dynamics damping="1000000.0" friction="0.0" />
+			<dynamics damping="${damping}" friction="0.0" />
 		</joint>
 		<link name="${name}">

File: urdf/lib/wheel/wheel.urdf.xacro (robot description, xacro)
@@ -1,5 +1,5 @@
 <?xml version="1.0"?>
 <robot name="wheel" xmlns:xacro="http://ros.org/wiki/xacro">
-	<xacro:macro name="wheel" params="name parent xyz:='0 0 0' rpy:='0 0 0'">
+	<xacro:macro name="wheel" params="name parent xyz:='0 0 0' rpy:='0 0 0' damping:=1000000.0">
 		<xacro:property name="radius" value="0.07825"/>
 		<xacro:property name="length" value="0.085"/>
@@ -11,5 +11,5 @@
 			<parent link="${parent}" />
 			<child link="${name}" />
-			<dynamics damping="1000000.0" friction="0.0" />
+			<dynamics damping="${damping}" friction="0.0" />
 		</joint>
 		<link name="${name}">

File: urdf/omni_wheel.urdf.xacro (robot description, xacro)
@@ -8,5 +8,5 @@
   </xacro:macro>
   <xacro:macro name="omni_wheel_250" params="name parent *origin">
-   <joint name="${name}_joint" type="fixed">
+   <joint name="${name}_joint" type="continuous">
     <xacro:insert_block name="origin" />
     <axis xyz="0 1 0" />
@@ -26,5 +26,5 @@
         <cylinder radius="0.07825" length="0.085"/>
      </geometry>
-     <material name="Neobotix/Black" />
+     <material name="Black" />
     </visual>
     <collision>
@@ -38,5 +38,5 @@
         <gravity>true</gravity>
         <self_collide>false</self_collide>
-        <material value="Gazebo/Black"/>
+        <material value="Black"/>
     </gazebo>
   </xacro:macro>

File: urdf/robot_dual_cam.urdf.xacro (robot description, xacro)
@@ -243,3 +243,71 @@
     </plugin>
   </gazebo>
+   <gazebo reference="agv_base_link">
+    <gravity>true</gravity>
+    <sensor name="imu_sensor" type="imu">
+      <always_on>true</always_on>
+      <update_rate>100</update_rate>
+      <visualize>true</visualize>
+      <topic>__default_topic__</topic>
+      <plugin filename="libgazebo_ros_imu_sensor.so" name="imu_plugin">
+        <topicName>imu</topicName>
+        <bodyName>imu_link</bodyName>
+        <updateRateHZ>10.0</updateRateHZ>
+        <gaussianNoise>0.0</gaussianNoise>
+        <xyzOffset>0 0 0</xyzOffset>
+        <rpyOffset>0 0 0</rpyOffset>
+        <frameName>imu_link</frameName>
+        <initialOrientationAsReference>false</initialOrientationAsReference>
+      </plugin>
+      <pose>0 0 0 0 0 0</pose>
+    </sensor>
+  </gazebo>
+<!--
+  <gazebo>
+  <plugin name="gazebo_ros_control" filename="libgazebo_ros_control.so">
+    <robotNamespace>/</robotNamespace>
+    <robotSimType>gazebo_ros_control/DefaultRobotHWSim</robotSimType>
+  </plugin>
+</gazebo>
+  <transmission name="tran1">
+    <type>transmission_interface/SimpleTransmission</type>
+    <joint name="wheel_front_left_joint">
+      <hardwareInterface>hardware_interface/VelocityJointInterface</hardwareInterface>
+    </joint>
+    <actuator name="motor1">
+      <hardwareInterface>VelocityJointInterface</hardwareInterface>
+      <mechanicalReduction>1</mechanicalReduction>
+    </actuator>
+  </transmission>
+  <transmission name="tran2">
+    <type>transmission_interface/SimpleTransmission</type>
+    <joint name="wheel_front_right_joint">
+      <hardwareInterface>VelocityJointInterface</hardwareInterface>
+    </joint>
+    <actuator name="motor2">
+      <hardwareInterface>VelocityJointInterface</hardwareInterface>
+      <mechanicalReduction>1</mechanicalReduction>
+    </actuator>
+  </transmission>
+  <transmission name="tran3">
+    <type>transmission_interface/SimpleTransmission</type>
+    <joint name="wheel_back_left_joint">
+      <hardwareInterface>hardware_interface/VelocityJointInterface</hardwareInterface>
+    </joint>
+    <actuator name="motor3">
+      <hardwareInterface>VelocityJointInterface</hardwareInterface>
+      <mechanicalReduction>1</mechanicalReduction>
+    </actuator>
+  </transmission>
+  <transmission name="tran4">
+    <type>transmission_interface/SimpleTransmission</type>
+    <joint name="wheel_back_right_joint">
+      <hardwareInterface>hardware_interface/VelocityJointInterface</hardwareInterface>
+    </joint>
+    <actuator name="motor4">
+      <hardwareInterface>VelocityJointInterface</hardwareInterface>
+      <mechanicalReduction>1</mechanicalReduction>
+    </actuator>
+  </transmission>
+ -->
 </robot>
